Commit message: Add dual-camera Isaac ROS pick-and-place simulation
Signed-off-by: 李博钊 <18622332179@163.com>

File: arx_r5_isaac_sim_bringup/urdf/r5a.isaac_sim.ros2_control.xacro (robot description, xacro)
@@ -86,5 +86,26 @@
         <state_interface name="velocity"/>
       </joint>
-      <!-- joint8 stays exclusively in the URDF/PhysX mimic relation. -->
+      <!--
+        joint8 is not claimed by a controller. TopicBasedSystem needs it in
+        the hardware block so its mimic pass can publish an eighth position
+        value matching the eighth joint name sent to Isaac Sim.
+      -->
+      <!--
+        Jazzy otherwise imports the robot URDF's mimic tag into ros2_control
+        and rejects this required transport command interface. Disable that
+        core mimic path here; TopicBasedSystem performs the explicit copy.
+      -->
+      <joint name="joint8" mimic="false">
+        <param name="mimic">joint7</param>
+        <param name="multiplier">1</param>
+        <command_interface name="position">
+          <param name="min">0.0</param>
+          <param name="max">0.044</param>
+        </command_interface>
+        <state_interface name="position">
+          <param name="initial_value">${initial_positions['joint8']}</param>
+        </state_interface>
+        <state_interface name="velocity"/>
+      </joint>
     </ros2_control>
   </xacro:macro>
